File: touchBoard/touchBoard.kicad_pcb (KiCad board)
At the start: 2 copper layers, 134.9 x 130 mm, 124 parts, among them J1 USB_C_16P, U1 ATSAMD21G18A-A, U2 AMS1117-3.3

Commit message: touchboard added leds
Parts:
- removed GND: GND, TestPoint:TestPoint_Pad_D1.5mm
- added D1: SK6812MINI, Library:LED_SK6812MINI_PLCC4_3.5x3.5mm_P1.75mm, B.Cu at (10.0, 10.0)
- added D10: SK6812MINI, Library:LED_SK6812MINI_PLCC4_3.5x3.5mm_P1.75mm, B.Cu at (20.0, 20.0)
- added D100: SK6812MINI, Library:LED_SK6812MINI_PLCC4_3.5x3.5mm_P1.75mm, B.Cu at (95.0, 27.5)
- added D101: SK6812MINI, Library:LED_SK6812MINI_PLCC4_3.5x3.5mm_P1.75mm, B.Cu at (95.0, 32.5)
- added D102: SK6812MINI, Library:LED_SK6812MINI_PLCC4_3.5x3.5mm_P1.75mm, B.Cu at (95.0, 37.5)
- added D103: SK6812MINI, Library:LED_SK6812MINI_PLCC4_3.5x3.5mm_P1.75mm, B.Cu at (95.0, 42.5)
- added D104: SK6812MINI, Library:LED_SK6812MINI_PLCC4_3.5x3.5mm_P1.75mm, B.Cu at (95.0, 47.5)
- added D105: SK6812MINI, Library:LED_SK6812MINI_PLCC4_3.5x3.5mm_P1.75mm, B.Cu at (95.0, 52.5)
- added D106: SK6812MINI, Library:LED_SK6812MINI_PLCC4_3.5x3.5mm_P1.75mm, B.Cu at (95.0, 57.5)
- added D107: SK6812MINI, Library:LED_SK6812MINI_PLCC4_3.5x3.5mm_P1.75mm, B.Cu at (110.0, 12.5)
- added D108: SK6812MINI, Library:LED_SK6812MINI_PLCC4_3.5x3.5mm_P1.75mm, B.Cu at (110.0, 17.5)
- added D109: SK6812MINI, Library:LED_SK6812MINI_PLCC4_3.5x3.5mm_P1.75mm, B.Cu at (110.0, 22.5)
- added D11: SK6812MINI, Library:LED_SK6812MINI_PLCC4_3.5x3.5mm_P1.75mm, B.Cu at (30.0, 20.0)
- added D110: SK6812MINI, Library:LED_SK6812MINI_PLCC4_3.5x3.5mm_P1.75mm, B.Cu at (110.0, 27.5)
- added D111: SK6812MINI, Library:LED_SK6812MINI_PLCC4_3.5x3.5mm_P1.75mm, B.Cu at (110.0, 32.5)
- added D112: SK6812MINI, Library:LED_SK6812MINI_PLCC4_3.5x3.5mm_P1.75mm, B.Cu at (110.0, 37.5)
- added D113: SK6812MINI, Library:LED_SK6812MINI_PLCC4_3.5x3.5mm_P1.75mm, B.Cu at (110.0, 42.5)
- added D114: SK6812MINI, Library:LED_SK6812MINI_PLCC4_3.5x3.5mm_P1.75mm, B.Cu at (110.0, 47.5)
- added D115: SK6812MINI, Library:LED_SK6812MINI_PLCC4_3.5x3.5mm_P1.75mm, B.Cu at (110.0, 52.5)
- added D116: SK6812MINI, Library:LED_SK6812MINI_PLCC4_3.5x3.5mm_P1.75mm, B.Cu at (110.0, 57.5)
- added D117: SK6812MINI, Library:LED_SK6812MINI_PLCC4_3.5x3.5mm_P1.75mm, B.Cu at (95.0, 72.5)
- added D118: SK6812MINI, Library:LED_SK6812MINI_PLCC4_3.5x3.5mm_P1.75mm, B.Cu at (95.0, 77.5)
- added D119: SK6812MINI, Library:LED_SK6812MINI_PLCC4_3.5x3.5mm_P1.75mm, B.Cu at (95.0, 82.5)
- added D12: SK6812MINI, Library:LED_SK6812MINI_PLCC4_3.5x3.5mm_P1.75mm, B.Cu at (40.0, 20.0)
- added D120: SK6812MINI, Library:LED_SK6812MINI_PLCC4_3.5x3.5mm_P1.75mm, B.Cu at (95.0, 87.5)
- added D121: SK6812MINI, Library:LED_SK6812MINI_PLCC4_3.5x3.5mm_P1.75mm, B.Cu at (95.0, 92.5)
- added D122: SK6812MINI, Library:LED_SK6812MINI_PLCC4_3.5x3.5mm_P1.75mm, B.Cu at (95.0, 97.5)
- added D123: SK6812MINI, Library:LED_SK6812MINI_PLCC4_3.5x3.5mm_P1.75mm, B.Cu at (95.0, 102.5)
- added D124: SK6812MINI, Library:LED_SK6812MINI_PLCC4_3.5x3.5mm_P1.75mm, B.Cu at (95.0, 107.5)
- added D125: SK6812MINI, Library:LED_SK6812MINI_PLCC4_3.5x3.5mm_P1.75mm, B.Cu at (95.0, 112.5)
- added D126: SK6812MINI, Library:LED_SK6812MINI_PLCC4_3.5x3.5mm_P1.75mm, B.Cu at (95.0, 117.5)
- added D127: SK6812MINI, Library:LED_SK6812MINI_PLCC4_3.5x3.5mm_P1.75mm, B.Cu at (110.0, 72.5)
- added D128: SK6812MINI, Library:LED_SK6812MINI_PLCC4_3.5x3.5mm_P1.75mm, B.Cu at (110.0, 77.5)
- added D129: SK6812MINI, Library:LED_SK6812MINI_PLCC4_3.5x3.5mm_P1.75mm, B.Cu at (110.0, 82.5)
- added D13: SK6812MINI, Library:LED_SK6812MINI_PLCC4_3.5x3.5mm_P1.75mm, B.Cu at (50.0, 20.0)
- added D130: SK6812MINI, Library:LED_SK6812MINI_PLCC4_3.5x3.5mm_P1.75mm, B.Cu at (110.0, 87.5)
- added D131: SK6812MINI, Library:LED_SK6812MINI_PLCC4_3.5x3.5mm_P1.75mm, B.Cu at (110.0, 92.5)
- added D132: SK6812MINI, Library:LED_SK6812MINI_PLCC4_3.5x3.5mm_P1.75mm, B.Cu at (110.0, 97.5)
- added D133: SK6812MINI, Library:LED_SK6812MINI_PLCC4_3.5x3.5mm_P1.75mm, B.Cu at (110.0, 102.5)
- added D134: SK6812MINI, Library:LED_SK6812MINI_PLCC4_3.5x3.5mm_P1.75mm, B.Cu at (110.0, 107.5)
- added D135: SK6812MINI, Library:LED_SK6812MINI_PLCC4_3.5x3.5mm_P1.75mm, B.Cu at (110.0, 112.5)
- added D136: SK6812MINI, Library:LED_SK6812MINI_PLCC4_3.5x3.5mm_P1.75mm, B.Cu at (110.0, 117.5)
- added D137: SK6812MINI, Library:LED_SK6812MINI_PLCC4_3.5x3.5mm_P1.75mm, B.Cu at (-8.50, 45.0)
- added D138: SK6812MINI, Library:LED_SK6812MINI_PLCC4_3.5x3.5mm_P1.75mm, B.Cu at (-2.50, 45.0)
- added D139: SK6812MINI, Library:LED_SK6812MINI_PLCC4_3.5x3.5mm_P1.75mm, B.Cu at (-8.50, 50.0)
- added D14: SK6812MINI, Library:LED_SK6812MINI_PLCC4_3.5x3.5mm_P1.75mm, B.Cu at (60.0, 20.0)
- added D140: SK6812MINI, Library:LED_SK6812MINI_PLCC4_3.5x3.5mm_P1.75mm, B.Cu at (-2.50, 50.0)
- added D141: SK6812MINI, Library:LED_SK6812MINI_PLCC4_3.5x3.5mm_P1.75mm, B.Cu at (-8.50, 55.0)
- added D142: SK6812MINI, Library:LED_SK6812MINI_PLCC4_3.5x3.5mm_P1.75mm, B.Cu at (-2.50, 55.0)
- added D143: SK6812MINI, Library:LED_SK6812MINI_PLCC4_3.5x3.5mm_P1.75mm, B.Cu at (-8.50, 60.0)
- added D144: SK6812MINI, Library:LED_SK6812MINI_PLCC4_3.5x3.5mm_P1.75mm, B.Cu at (-2.50, 60.0)
- added D145: SK6812MINI, Library:LED_SK6812MINI_PLCC4_3.5x3.5mm_P1.75mm, B.Cu at (-8.50, 65.0)
- added D146: SK6812MINI, Library:LED_SK6812MINI_PLCC4_3.5x3.5mm_P1.75mm, B.Cu at (-2.50, 65.0)
- added D147: SK6812MINI, Library:LED_SK6812MINI_PLCC4_3.5x3.5mm_P1.75mm, B.Cu at (-8.50, 70.0)
- added D148: SK6812MINI, Library:LED_SK6812MINI_PLCC4_3.5x3.5mm_P1.75mm, B.Cu at (-2.50, 70.0)
- added D149: SK6812MINI, Library:LED_SK6812MINI_PLCC4_3.5x3.5mm_P1.75mm, B.Cu at (-8.50, 75.0)
- added D15: SK6812MINI, Library:LED_SK6812MINI_PLCC4_3.5x3.5mm_P1.75mm, B.Cu at (70.0, 20.0)
- added D150: SK6812MINI, Library:LED_SK6812MINI_PLCC4_3.5x3.5mm_P1.75mm, B.Cu at (-2.50, 75.0)
- added D151: SK6812MINI, Library:LED_SK6812MINI_PLCC4_3.5x3.5mm_P1.75mm, B.Cu at (-8.50, 80.0)
- added D152: SK6812MINI, Library:LED_SK6812MINI_PLCC4_3.5x3.5mm_P1.75mm, B.Cu at (-2.50, 80.0)
- added D153: SK6812MINI, Library:LED_SK6812MINI_PLCC4_3.5x3.5mm_P1.75mm, B.Cu at (-8.50, 85.0)
- added D154: SK6812MINI, Library:LED_SK6812MINI_PLCC4_3.5x3.5mm_P1.75mm, B.Cu at (-2.50, 85.0)
- added D155: SK6812MINI, Library:LED_SK6812MINI_PLCC4_3.5x3.5mm_P1.75mm, B.Cu at (-8.50, 90.0)
- added D156: SK6812MINI, Library:LED_SK6812MINI_PLCC4_3.5x3.5mm_P1.75mm, B.Cu at (-2.50, 90.0)
- added D157: SK6812MINI, Library:LED_SK6812MINI_PLCC4_3.5x3.5mm_P1.75mm, B.Cu at (-8.50, 95.0)
- added D158: SK6812MINI, Library:LED_SK6812MINI_PLCC4_3.5x3.5mm_P1.75mm, B.Cu at (-2.50, 95.0)
- added D159: SK6812MINI, Library:LED_SK6812MINI_PLCC4_3.5x3.5mm_P1.75mm, B.Cu at (-8.50, 100.0)
- added D16: SK6812MINI, Library:LED_SK6812MINI_PLCC4_3.5x3.5mm_P1.75mm, B.Cu at (80.0, 20.0)
- added D160: SK6812MINI, Library:LED_SK6812MINI_PLCC4_3.5x3.5mm_P1.75mm, B.Cu at (-2.50, 100.0)
- added D161: SK6812MINI, Library:LED_SK6812MINI_PLCC4_3.5x3.5mm_P1.75mm, B.Cu at (-8.50, 105.0)
- added D162: SK6812MINI, Library:LED_SK6812MINI_PLCC4_3.5x3.5mm_P1.75mm, B.Cu at (-2.50, 105.0)
- added D163: SK6812MINI, Library:LED_SK6812MINI_PLCC4_3.5x3.5mm_P1.75mm, B.Cu at (-8.50, 110.0)
- added D164: SK6812MINI, Library:LED_SK6812MINI_PLCC4_3.5x3.5mm_P1.75mm, B.Cu at (-2.50, 110.0)
- added D17: SK6812MINI, Library:LED_SK6812MINI_PLCC4_3.5x3.5mm_P1.75mm, B.Cu at (10.0, 30.0)
- added D18: SK6812MINI, Library:LED_SK6812MINI_PLCC4_3.5x3.5mm_P1.75mm, B.Cu at (20.0, 30.0)
- added D19: SK6812MINI, Library:LED_SK6812MINI_PLCC4_3.5x3.5mm_P1.75mm, B.Cu at (30.0, 30.0)
- added D2: SK6812MINI, Library:LED_SK6812MINI_PLCC4_3.5x3.5mm_P1.75mm, B.Cu at (20.0, 10.0)
- added D20: SK6812MINI, Library:LED_SK6812MINI_PLCC4_3.5x3.5mm_P1.75mm, B.Cu at (40.0, 30.0)
- added D21: SK6812MINI, Library:LED_SK6812MINI_PLCC4_3.5x3.5mm_P1.75mm, B.Cu at (50.0, 30.0)
- added D22: SK6812MINI, Library:LED_SK6812MINI_PLCC4_3.5x3.5mm_P1.75mm, B.Cu at (60.0, 30.0)
- added D23: SK6812MINI, Library:LED_SK6812MINI_PLCC4_3.5x3.5mm_P1.75mm, B.Cu at (70.0, 30.0)
- added D24: SK6812MINI, Library:LED_SK6812MINI_PLCC4_3.5x3.5mm_P1.75mm, B.Cu at (80.0, 30.0)
- added D25: SK6812MINI, Library:LED_SK6812MINI_PLCC4_3.5x3.5mm_P1.75mm, B.Cu at (10.0, 40.0)
- added D26: SK6812MINI, Library:LED_SK6812MINI_PLCC4_3.5x3.5mm_P1.75mm, B.Cu at (20.0, 40.0)
- added D27: SK6812MINI, Library:LED_SK6812MINI_PLCC4_3.5x3.5mm_P1.75mm, B.Cu at (30.0, 40.0)
- added D28: SK6812MINI, Library:LED_SK6812MINI_PLCC4_3.5x3.5mm_P1.75mm, B.Cu at (40.0, 40.0)
- added D29: SK6812MINI, Library:LED_SK6812MINI_PLCC4_3.5x3.5mm_P1.75mm, B.Cu at (50.0, 40.0)
- added D3: SK6812MINI, Library:LED_SK6812MINI_PLCC4_3.5x3.5mm_P1.75mm, B.Cu at (30.0, 10.0)
- added D30: SK6812MINI, Library:LED_SK6812MINI_PLCC4_3.5x3.5mm_P1.75mm, B.Cu at (60.0, 40.0)
- added D31: SK6812MINI, Library:LED_SK6812MINI_PLCC4_3.5x3.5mm_P1.75mm, B.Cu at (70.0, 40.0)
- added D32: SK6812MINI, Library:LED_SK6812MINI_PLCC4_3.5x3.5mm_P1.75mm, B.Cu at (80.0, 40.0)
- added D33: SK6812MINI, Library:LED_SK6812MINI_PLCC4_3.5x3.5mm_P1.75mm, B.Cu at (10.0, 50.0)
- added D34: SK6812MINI, Library:LED_SK6812MINI_PLCC4_3.5x3.5mm_P1.75mm, B.Cu at (20.0, 50.0)
- added D35: SK6812MINI, Library:LED_SK6812MINI_PLCC4_3.5x3.5mm_P1.75mm, B.Cu at (30.0, 50.0)
- added D36: SK6812MINI, Library:LED_SK6812MINI_PLCC4_3.5x3.5mm_P1.75mm, B.Cu at (40.0, 50.0)
- added D37: SK6812MINI, Library:LED_SK6812MINI_PLCC4_3.5x3.5mm_P1.75mm, B.Cu at (50.0, 50.0)
- added D38: SK6812MINI, Library:LED_SK6812MINI_PLCC4_3.5x3.5mm_P1.75mm, B.Cu at (60.0, 50.0)
- added D39: SK6812MINI, Library:LED_SK6812MINI_PLCC4_3.5x3.5mm_P1.75mm, B.Cu at (70.0, 50.0)
- added D4: SK6812MINI, Library:LED_SK6812MINI_PLCC4_3.5x3.5mm_P1.75mm, B.Cu at (40.0, 10.0)
- added D40: SK6812MINI, Library:LED_SK6812MINI_PLCC4_3.5x3.5mm_P1.75mm, B.Cu at (80.0, 50.0)
- added D41: SK6812MINI, Library:LED_SK6812MINI_PLCC4_3.5x3.5mm_P1.75mm, B.Cu at (10.0, 60.0)
- added D42: SK6812MINI, Library:LED_SK6812MINI_PLCC4_3.5x3.5mm_P1.75mm, B.Cu at (20.0, 60.0)
- added D43: SK6812MINI, Library:LED_SK6812MINI_PLCC4_3.5x3.5mm_P1.75mm, B.Cu at (30.0, 60.0)
- added D44: SK6812MINI, Library:LED_SK6812MINI_PLCC4_3.5x3.5mm_P1.75mm, B.Cu at (40.0, 60.0)
- added D45: SK6812MINI, Library:LED_SK6812MINI_PLCC4_3.5x3.5mm_P1.75mm, B.Cu at (50.0, 60.0)
- added D46: SK6812MINI, Library:LED_SK6812MINI_PLCC4_3.5x3.5mm_P1.75mm, B.Cu at (60.0, 60.0)
- added D47: SK6812MINI, Library:LED_SK6812MINI_PLCC4_3.5x3.5mm_P1.75mm, B.Cu at (70.0, 60.0)
- added D48: SK6812MINI, Library:LED_SK6812MINI_PLCC4_3.5x3.5mm_P1.75mm, B.Cu at (80.0, 60.0)
- added D49: SK6812MINI, Library:LED_SK6812MINI_PLCC4_3.5x3.5mm_P1.75mm, B.Cu at (10.0, 70.0)
- added D5: SK6812MINI, Library:LED_SK6812MINI_PLCC4_3.5x3.5mm_P1.75mm, B.Cu at (50.0, 10.0)
- added D50: SK6812MINI, Library:LED_SK6812MINI_PLCC4_3.5x3.5mm_P1.75mm, B.Cu at (20.0, 70.0)
- added D51: SK6812MINI, Library:LED_SK6812MINI_PLCC4_3.5x3.5mm_P1.75mm, B.Cu at (30.0, 70.0)
- added D52: SK6812MINI, Library:LED_SK6812MINI_PLCC4_3.5x3.5mm_P1.75mm, B.Cu at (40.0, 70.0)
- added D53: SK6812MINI, Library:LED_SK6812MINI_PLCC4_3.5x3.5mm_P1.75mm, B.Cu at (50.0, 70.0)
- added D54: SK6812MINI, Library:LED_SK6812MINI_PLCC4_3.5x3.5mm_P1.75mm, B.Cu at (60.0, 70.0)
- added D55: SK6812MINI, Library:LED_SK6812MINI_PLCC4_3.5x3.5mm_P1.75mm, B.Cu at (70.0, 70.0)
- added D56: SK6812MINI, Library:LED_SK6812MINI_PLCC4_3.5x3.5mm_P1.75mm, B.Cu at (80.0, 70.0)
- added D57: SK6812MINI, Library:LED_SK6812MINI_PLCC4_3.5x3.5mm_P1.75mm, B.Cu at (10.0, 80.0)
- added D58: SK6812MINI, Library:LED_SK6812MINI_PLCC4_3.5x3.5mm_P1.75mm, B.Cu at (20.0, 80.0)
- added D59: SK6812MINI, Library:LED_SK6812MINI_PLCC4_3.5x3.5mm_P1.75mm, B.Cu at (30.0, 80.0)
- added D6: SK6812MINI, Library:LED_SK6812MINI_PLCC4_3.5x3.5mm_P1.75mm, B.Cu at (60.0, 10.0)
- added D60: SK6812MINI, Library:LED_SK6812MINI_PLCC4_3.5x3.5mm_P1.75mm, B.Cu at (40.0, 80.0)
- added D61: SK6812MINI, Library:LED_SK6812MINI_PLCC4_3.5x3.5mm_P1.75mm, B.Cu at (50.0, 80.0)
- added D62: SK6812MINI, Library:LED_SK6812MINI_PLCC4_3.5x3.5mm_P1.75mm, B.Cu at (60.0, 80.0)
- added D63: SK6812MINI, Library:LED_SK6812MINI_PLCC4_3.5x3.5mm_P1.75mm, B.Cu at (70.0, 80.0)
- added D64: SK6812MINI, Library:LED_SK6812MINI_PLCC4_3.5x3.5mm_P1.75mm, B.Cu at (80.0, 80.0)
- added D65: SK6812MINI, Library:LED_SK6812MINI_PLCC4_3.5x3.5mm_P1.75mm, B.Cu at (10.0, 90.0)
- added D66: SK6812MINI, Library:LED_SK6812MINI_PLCC4_3.5x3.5mm_P1.75mm, B.Cu at (20.0, 90.0)
- added D67: SK6812MINI, Library:LED_SK6812MINI_PLCC4_3.5x3.5mm_P1.75mm, B.Cu at (30.0, 90.0)
- added D68: SK6812MINI, Library:LED_SK6812MINI_PLCC4_3.5x3.5mm_P1.75mm, B.Cu at (40.0, 90.0)
- added D69: SK6812MINI, Library:LED_SK6812MINI_PLCC4_3.5x3.5mm_P1.75mm, B.Cu at (50.0, 90.0)
- added D7: SK6812MINI, Library:LED_SK6812MINI_PLCC4_3.5x3.5mm_P1.75mm, B.Cu at (70.0, 10.0)
- added D70: SK6812MINI, Library:LED_SK6812MINI_PLCC4_3.5x3.5mm_P1.75mm, B.Cu at (60.0, 90.0)
- added D71: SK6812MINI, Library:LED_SK6812MINI_PLCC4_3.5x3.5mm_P1.75mm, B.Cu at (70.0, 90.0)
- added D72: SK6812MINI, Library:LED_SK6812MINI_PLCC4_3.5x3.5mm_P1.75mm, B.Cu at (80.0, 90.0)
- added D73: SK6812MINI, Library:LED_SK6812MINI_PLCC4_3.5x3.5mm_P1.75mm, B.Cu at (10.0, 100.0)
- added D74: SK6812MINI, Library:LED_SK6812MINI_PLCC4_3.5x3.5mm_P1.75mm, B.Cu at (20.0, 100.0)
- added D75: SK6812MINI, Library:LED_SK6812MINI_PLCC4_3.5x3.5mm_P1.75mm, B.Cu at (30.0, 100.0)
- added D76: SK6812MINI, Library:LED_SK6812MINI_PLCC4_3.5x3.5mm_P1.75mm, B.Cu at (40.0, 100.0)
- added D77: SK6812MINI, Library:LED_SK6812MINI_PLCC4_3.5x3.5mm_P1.75mm, B.Cu at (50.0, 100.0)
- added D78: SK6812MINI, Library:LED_SK6812MINI_PLCC4_3.5x3.5mm_P1.75mm, B.Cu at (60.0, 100.0)
- added D79: SK6812MINI, Library:LED_SK6812MINI_PLCC4_3.5x3.5mm_P1.75mm, B.Cu at (70.0, 100.0)
- added D8: SK6812MINI, Library:LED_SK6812MINI_PLCC4_3.5x3.5mm_P1.75mm, B.Cu at (80.0, 10.0)
- added D80: SK6812MINI, Library:LED_SK6812MINI_PLCC4_3.5x3.5mm_P1.75mm, B.Cu at (80.0, 100.0)
- added D81: SK6812MINI, Library:LED_SK6812MINI_PLCC4_3.5x3.5mm_P1.75mm, B.Cu at (10.0, 110.0)
- added D82: SK6812MINI, Library:LED_SK6812MINI_PLCC4_3.5x3.5mm_P1.75mm, B.Cu at (20.0, 110.0)
- added D83: SK6812MINI, Library:LED_SK6812MINI_PLCC4_3.5x3.5mm_P1.75mm, B.Cu at (30.0, 110.0)
- added D84: SK6812MINI, Library:LED_SK6812MINI_PLCC4_3.5x3.5mm_P1.75mm, B.Cu at (40.0, 110.0)
- added D85: SK6812MINI, Library:LED_SK6812MINI_PLCC4_3.5x3.5mm_P1.75mm, B.Cu at (50.0, 110.0)
- added D86: SK6812MINI, Library:LED_SK6812MINI_PLCC4_3.5x3.5mm_P1.75mm, B.Cu at (60.0, 110.0)
- added D87: SK6812MINI, Library:LED_SK6812MINI_PLCC4_3.5x3.5mm_P1.75mm, B.Cu at (70.0, 110.0)
- added D88: SK6812MINI, Library:LED_SK6812MINI_PLCC4_3.5x3.5mm_P1.75mm, B.Cu at (80.0, 110.0)
- added D89: SK6812MINI, Library:LED_SK6812MINI_PLCC4_3.5x3.5mm_P1.75mm, B.Cu at (10.0, 120.0)
- added D9: SK6812MINI, Library:LED_SK6812MINI_PLCC4_3.5x3.5mm_P1.75mm, B.Cu at (10.0, 20.0)
- added D90: SK6812MINI, Library:LED_SK6812MINI_PLCC4_3.5x3.5mm_P1.75mm, B.Cu at (20.0, 120.0)
- added D91: SK6812MINI, Library:LED_SK6812MINI_PLCC4_3.5x3.5mm_P1.75mm, B.Cu at (30.0, 120.0)
- added D92: SK6812MINI, Library:LED_SK6812MINI_PLCC4_3.5x3.5mm_P1.75mm, B.Cu at (40.0, 120.0)
- added D93: SK6812MINI, Library:LED_SK6812MINI_PLCC4_3.5x3.5mm_P1.75mm, B.Cu at (50.0, 120.0)
- added D94: SK6812MINI, Library:LED_SK6812MINI_PLCC4_3.5x3.5mm_P1.75mm, B.Cu at (60.0, 120.0)
- added D95: SK6812MINI, Library:LED_SK6812MINI_PLCC4_3.5x3.5mm_P1.75mm, B.Cu at (70.0, 120.0)
- added D96: SK6812MINI, Library:LED_SK6812MINI_PLCC4_3.5x3.5mm_P1.75mm, B.Cu at (80.0, 120.0)
- added D97: SK6812MINI, Library:LED_SK6812MINI_PLCC4_3.5x3.5mm_P1.75mm, B.Cu at (95.0, 12.5)
- added D98: SK6812MINI, Library:LED_SK6812MINI_PLCC4_3.5x3.5mm_P1.75mm, B.Cu at (95.0, 17.5)
- added D99: SK6812MINI, Library:LED_SK6812MINI_PLCC4_3.5x3.5mm_P1.75mm, B.Cu at (95.0, 22.5)
- added REF**: MountingHole_3.2mm_M3, MountingHole:MountingHole_3.2mm_M3, F.Cu at (116.0, 4.00)
- added REF**: MountingHole_3.2mm_M3, MountingHole:MountingHole_3.2mm_M3, F.Cu at (-9.00, 126.0)
- added REF**: MountingHole_3.2mm_M3, MountingHole:MountingHole_3.2mm_M3, F.Cu at (-9.00, 4.00)
- added REF**: MountingHole_3.2mm_M3, MountingHole:MountingHole_3.2mm_M3, F.Cu at (116.0, 126.0)
- added TP4: GND, TestPoint:TestPoint_Pad_D1.5mm, F.Cu at (-11.0, 11.5)
- TP10: value TestPoint -> MISO
- TP11: value TestPoint -> LED
- TP5: value TestPoint -> USB_D+
- TP6: value TestPoint -> USB_D-
- TP7: value TestPoint -> CS
- TP8: value TestPoint -> SCLK
- TP9: value TestPoint -> MOSI
- moved TP6 55.0 mm to (2.00, 4.00), turned to 90 degrees
- moved TP5 49.8 mm to (-2.00, 4.00), turned to 90 degrees
- moved TP11 47.9 mm to (-11.0, 23.0)
- moved TP10 40.9 mm to (-11.0, 27.0)
- moved TP9 35.5 mm to (-11.0, 29.5)
- moved TP8 30.3 mm to (-11.0, 32.0)
- moved TP7 25.5 mm to (-11.0, 34.5)
- moved C5 3.00 mm to (-1.00, 11.5)
- moved C6 3.00 mm to (-1.00, 13.5)
- moved L1 3.00 mm to (-1.00, 15.5)
- moved R1 3.00 mm to (-4.00, 14.5)
- moved C7 2.92 mm to (-6.50, 38.5), turned to 0 degrees
- moved C8 2.92 mm to (-6.50, 40.5), turned to 0 degrees
- moved U2 2.92 mm to (-5.50, 33.5)
- moved C1 2.24 mm to (-8.00, 23.0)
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Routing:
- net +5V: track 57.0 -> 962.8 mm, vias 0 -> 2
- net Net-(D96-DOUT): track 0.00 -> 114.8 mm, vias 0 -> 2
- net Net-(D16-DOUT): track 0.00 -> 91.2 mm, vias 0 -> 2
- net Net-(D24-DOUT): track 0.00 -> 91.0 mm, vias 0 -> 2
- net Net-(D88-DOUT): track 0.00 -> 90.6 mm, vias 0 -> 2
- net Net-(D80-DOUT): track 0.00 -> 90.6 mm, vias 0 -> 2
- net Net-(D72-DOUT): track 0.00 -> 90.6 mm, vias 0 -> 2
- net Net-(D64-DOUT): track 0.00 -> 90.6 mm, vias 0 -> 2
- net Net-(D56-DOUT): track 0.00 -> 90.6 mm, vias 0 -> 2
- net Net-(D48-DOUT): track 0.00 -> 90.6 mm, vias 0 -> 2
- net Net-(D40-DOUT): track 0.00 -> 90.6 mm, vias 0 -> 2
- net Net-(D32-DOUT): track 0.00 -> 90.6 mm, vias 0 -> 2
- net Net-(D8-DOUT): track 0.00 -> 84.5 mm
- net CS: track 0.00 -> 18.1 mm, vias 0 -> 1
- net SCLK: track 0.00 -> 17.3 mm, vias 0 -> 1
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Other:
- board size 134.9 x 130 mm -> 132.9 x 130 mm
