File: touchBoard/touchBoard.kicad_sch (KiCad schematic)
At the start: 131 parts, among them J1 USB_C_16P, U1 ATSAMD21G18A-A

Commit message: created touch board
Parts:
- removed TP3: TestPoint_Alt, symbol Connector:TestPoint_Alt
- removed Touch100, Touch101, Touch102, Touch103, Touch104, Touch105, Touch106, Touch107, Touch108, Touch109, Touch110, Touch111, Touch112, Touch113, Touch114, Touch115, Touch116, Touch117, Touch118, Touch119, Touch120, Touch97, Touch98, Touch99: TestPoint_2Pole, symbol Connector:TestPoint_2Pole
- added C7: 10uF, Capacitor_SMD:C_0805_2012Metric_Pad1.18x1.45mm_HandSolder, symbol Device:C
- added C8: 100nF, Capacitor_SMD:C_0805_2012Metric_Pad1.18x1.45mm_HandSolder, symbol Device:C
- added R1: 1k, Resistor_SMD:R_0805_2012Metric_Pad1.20x1.40mm_HandSolder, symbol Device:R
- added TP10, TP11, TP2, TP3, TP4, TP5, TP6, TP7, TP8, TP9: TestPoint, TestPoint:TestPoint_Pad_D1.5mm, symbol Connector:TestPoint
- added TS1, TS2, TS3, TS4: ~, Library:TouchSlider, symbol Library:TouchSlider
- added U2: AMS1117-3.3, Package_TO_SOT_SMD:SOT-223-3_TabPin2, symbol Regulator_Linear:AMS1117-3.3
- C1, C2, C3, C4, C5, C6: footprint (none) -> Capacitor_SMD:C_0805_2012Metric_Pad1.18x1.45mm_HandSolder
- J1: footprint (none) -> Connector_USB:USB_C_Receptacle_HCTL_HC-TYPE-C-16P-01A
- L1: footprint (none) -> Inductor_SMD:L_0805_2012Metric_Pad1.15x1.40mm_HandSolder
- TP1: footprint (none) -> TestPoint:TestPoint_Pad_D1.5mm
- Touch1, Touch10, Touch11, Touch12, Touch13, Touch14, Touch15, Touch16, Touch17, Touch18, Touch19, Touch2, Touch20, Touch21, Touch22, Touch23, Touch24, Touch25, Touch26, Touch27, Touch28, Touch29, Touch3, Touch30, Touch31, Touch32, Touch33, Touch34, Touch35, Touch36, Touch37, Touch38, Touch39, Touch4, Touch40, Touch41, Touch42, Touch43, Touch44, Touch45, Touch46, Touch47, Touch48, Touch49, Touch5, Touch50, Touch51, Touch52, Touch53, Touch54, Touch55, Touch56, Touch57, Touch58, Touch59, Touch6, Touch60, Touch61, Touch62, Touch63, Touch64, Touch65, Touch66, Touch67, Touch68, Touch69, Touch7, Touch70, Touch71, Touch72, Touch73, Touch74, Touch75, Touch76, Touch77, Touch78, Touch79, Touch8, Touch80, Touch81, Touch82, Touch83, Touch84, Touch85, Touch86, Touch87, Touch88, Touch89, Touch9, Touch90, Touch91, Touch92, Touch93, Touch94, Touch95, Touch96: footprint (none) -> Library:TouchButton
Connections:
- net +3V3: now also R1.2, U2.2 (VO)
- net +5V: now also C7.1, C8.1, U2.3 (VI)
- net GND: now also C7.2, C8.2, TP4.1, U2.1 (GND)
- net RST: now also TP1.1
- net SWCLK: now also R1.1, TP3.1
- net SWDIO: now also TP2.1
- net USB_D+: now also TP5.1
- net USB_D-: now also TP6.1
- net X0: now also TS1.1 (X1), TS2.1 (X1); no longer Touch10.1, Touch9.1
- net X1: now also Touch10.1, Touch9.1, TS1.2 (X2), TS2.2 (X2); no longer Touch17.1, Touch18.1, Touch19.1, Touch20.1
- net X10: now also Touch81.1, Touch82.1, Touch83.1, Touch84.1, Touch85.1, Touch86.1, Touch87.1, Touch88.1, TS3.5 (X5), TS4.5 (X5)
- net X11: now also Touch89.1, Touch90.1, Touch91.1, Touch92.1, Touch93.1, Touch94.1, Touch95.1, Touch96.1, TS3.6 (X6), TS4.6 (X6)
- net X2: now also Touch17.1, Touch18.1, Touch19.1, Touch20.1, TS1.3 (X3), TS2.3 (X3); no longer Touch25.1, Touch26.1, Touch27.1, Touch28.1, Touch29.1, Touch30.1
- net X3: now also Touch25.1, Touch26.1, Touch27.1, Touch28.1, Touch29.1, Touch30.1, TS1.4 (X4), TS2.4 (X4); no longer Touch33.1, Touch34.1, Touch35.1, Touch36.1, Touch37.1, Touch38.1, Touch39.1, Touch40.1
- net X4: now also Touch33.1, Touch34.1, Touch35.1, Touch36.1, Touch37.1, Touch38.1, Touch39.1, Touch40.1, TS1.5 (X5), TS2.5 (X5); no longer Touch41.1, Touch42.1, Touch43.1, Touch44.1, Touch45.1, Touch46.1, Touch47.1, Touch48.1, Touch49.1, Touch50.1
- net X5: now also Touch41.1, Touch42.1, Touch43.1, Touch44.1, Touch45.1, Touch46.1, Touch47.1, Touch48.1, TS1.6 (X6), TS2.6 (X6); no longer Touch51.1, Touch52.1, Touch53.1, Touch54.1, Touch55.1, Touch56.1, Touch57.1, Touch58.1, Touch59.1, Touch60.1
- net X6: now also Touch49.1, Touch50.1, Touch51.1, Touch52.1, Touch53.1, Touch54.1, Touch55.1, Touch56.1, TS3.1 (X1), TS4.1 (X1); no longer Touch61.1, Touch62.1, Touch63.1, Touch64.1, Touch65.1, Touch66.1, Touch67.1, Touch68.1, Touch69.1, Touch70.1
- net X7: now also Touch57.1, Touch58.1, Touch59.1, Touch60.1, Touch61.1, Touch62.1, Touch63.1, Touch64.1, TS3.2 (X2), TS4.2 (X2); no longer Touch71.1, Touch72.1, Touch73.1, Touch74.1, Touch75.1, Touch76.1, Touch77.1, Touch78.1, Touch79.1, Touch80.1
- net X8: now also Touch65.1, Touch66.1, Touch67.1, Touch68.1, Touch69.1, Touch70.1, Touch71.1, Touch72.1, TS3.3 (X3), TS4.3 (X3); no longer Touch81.1, Touch82.1, Touch83.1, Touch84.1, Touch85.1, Touch86.1, Touch87.1, Touch88.1, Touch89.1, Touch90.1
- net X9: now also Touch73.1, Touch74.1, Touch75.1, Touch76.1, Touch77.1, Touch78.1, Touch79.1, Touch80.1, TS3.4 (X4), TS4.4 (X4); no longer Touch91.1, Touch92.1, Touch93.1, Touch94.1, Touch95.1, Touch96.1
- net Y0: now also Touch17.2, Touch25.2, Touch33.2, Touch49.2, Touch57.2, Touch65.2, Touch73.2, Touch89.2, Touch9.2; no longer Touch11.2, Touch21.2, Touch31.2, Touch51.2, Touch61.2, Touch71.2, Touch91.2
- net Y1: now also Touch10.2, Touch18.2, Touch26.2, Touch34.2, Touch50.2, Touch58.2, Touch66.2, Touch74.2, Touch90.2; no longer Touch12.2, Touch22.2, Touch32.2, Touch52.2, Touch62.2, Touch72.2, Touch92.2
- net Y14: now also TS1.0 (Y), TS3.0 (Y); no longer Touch19.2, Touch29.2, Touch39.2, Touch49.2, Touch59.2, Touch69.2, Touch79.2, Touch89.2, Touch9.2
- net Y15: now also TS2.0 (Y), TS4.0 (Y); no longer Touch10.2, Touch20.2, Touch30.2, Touch40.2, Touch50.2, Touch60.2, Touch70.2, Touch80.2, Touch90.2
- net Y2: now also Touch11.2, Touch19.2, Touch27.2, Touch35.2, Touch51.2, Touch59.2, Touch67.2, Touch75.2, Touch91.2; no longer Touch13.2, Touch23.2, Touch33.2, Touch53.2, Touch63.2, Touch73.2, Touch93.2
- net Y3: now also Touch12.2, Touch20.2, Touch28.2, Touch36.2, Touch52.2, Touch60.2, Touch68.2, Touch76.2, Touch92.2; no longer Touch14.2, Touch24.2, Touch34.2, Touch54.2, Touch64.2, Touch74.2, Touch94.2
- net Y4: now also Touch13.2, Touch21.2, Touch29.2, Touch37.2, Touch53.2, Touch61.2, Touch69.2, Touch77.2, Touch93.2; no longer Touch15.2, Touch25.2, Touch35.2, Touch55.2, Touch65.2, Touch75.2, Touch95.2
- net Y5: now also Touch14.2, Touch22.2, Touch30.2, Touch38.2, Touch54.2, Touch62.2, Touch70.2, Touch78.2, Touch94.2; no longer Touch16.2, Touch26.2, Touch36.2, Touch56.2, Touch66.2, Touch76.2, Touch96.2
- net Y8: now also Touch15.2, Touch23.2, Touch31.2, Touch39.2, Touch55.2, Touch63.2, Touch71.2, Touch79.2, Touch95.2; no longer Touch17.2, Touch27.2, Touch37.2, Touch57.2, Touch67.2, Touch77.2
- net Y9: now also Touch16.2, Touch24.2, Touch32.2, Touch40.2, Touch56.2, Touch64.2, Touch72.2, Touch80.2, Touch96.2; no longer Touch18.2, Touch28.2, Touch38.2, Touch58.2, Touch68.2, Touch78.2
- net CC1: now reaches J1.A5 (CC1)
- net CC2: now reaches J1.B5 (CC2)
- net MISO: now reaches U1.21 (PA12)
- net MISO: now also TP10.1
- net MOSI: now reaches U1.22 (PA13)
- net MOSI: now also TP9.1
- net SCLK: now reaches U1.23 (PA14)
- net SCLK: now also TP8.1
- net CS: now reaches U1.24 (PA15)
- net CS: now also TP7.1
- net LED: now reaches U1.37 (PB22)
- net LED: now also TP11.1
- no-connect marks 8 -> 7
Other:
- moved on the sheet: TP1

Commit message: touchboard added leds
Parts:
- added D1, D10, D100, D101, D102, D103, D104, D105, D106, D107, D108, D109, D11, D110, D111, D112, D113, D114, D115, D116, D117, D118, D119, D12, D120, D121, D122, D123, D124, D125, D126, D127, D128, D129, D13, D130, D131, D132, D133, D134, D135, D136, D137, D138, D139, D14, D140, D141, D142, D143, D144, D145, D146, D147, D148, D149, D15, D150, D151, D152, D153, D154, D155, D156, D157, D158, D159, D16, D160, D161, D162, D163, D164, D17, D18, D19, D2, D20, D21, D22, D23, D24, D25, D26, D27, D28, D29, D3, D30, D31, D32, D33, D34, D35, D36, D37, D38, D39, D4, D40, D41, D42, D43, D44, D45, D46, D47, D48, D49, D5, D50, D51, D52, D53, D54, D55, D56, D57, D58, D59, D6, D60, D61, D62, D63, D64, D65, D66, D67, D68, D69, D7, D70, D71, D72, D73, D74, D75, D76, D77, D78, D79, D8, D80, D81, D82, D83, D84, D85, D86, D87, D88, D89, D9, D90, D91, D92, D93, D94, D95, D96, D97, D98, D99: SK6812MINI, Library:LED_SK6812MINI_PLCC4_3.5x3.5mm_P1.75mm, symbol LED:SK6812MINI
- TP1: value TestPoint -> RST
- TP10: value TestPoint -> MISO
- TP11: value TestPoint -> LED
- TP2: value TestPoint -> SWDIO
- TP3: value TestPoint -> SWCLK
- TP4: value TestPoint -> GND
- TP5: value TestPoint -> USB_D+
- TP6: value TestPoint -> USB_D-
- TP7: value TestPoint -> CS
- TP8: value TestPoint -> SCLK
- TP9: value TestPoint -> MOSI
Connections:
- net +5V: now also D1.4 (VDD), D10.4 (VDD), D100.4 (VDD), D101.4 (VDD), D102.4 (VDD), D103.4 (VDD), D104.4 (VDD), D105.4 (VDD), D106.4 (VDD), D107.4 (VDD), D108.4 (VDD), D109.4 (VDD), D11.4 (VDD), D110.4 (VDD), D111.4 (VDD), D112.4 (VDD), D113.4 (VDD), D114.4 (VDD), D115.4 (VDD), D116.4 (VDD), D117.4 (VDD), D118.4 (VDD), D119.4 (VDD), D12.4 (VDD), D120.4 (VDD), D121.4 (VDD), D122.4 (VDD), D123.4 (VDD), D124.4 (VDD), D125.4 (VDD), D126.4 (VDD), D127.4 (VDD), D128.4 (VDD), D129.4 (VDD), D13.4 (VDD), D130.4 (VDD), D131.4 (VDD), D132.4 (VDD), D133.4 (VDD), D134.4 (VDD), D135.4 (VDD), D136.4 (VDD), D137.4 (VDD), D138.4 (VDD), D139.4 (VDD), D14.4 (VDD), D140.4 (VDD), D141.4 (VDD), D142.4 (VDD), D143.4 (VDD), D144.4 (VDD), D145.4 (VDD), D146.4 (VDD), D147.4 (VDD), D148.4 (VDD), D149.4 (VDD), D15.4 (VDD), D150.4 (VDD), D151.4 (VDD), D152.4 (VDD), D153.4 (VDD), D154.4 (VDD), D155.4 (VDD), D156.4 (VDD), D157.4 (VDD), D158.4 (VDD), D159.4 (VDD), D16.4 (VDD), D160.4 (VDD), D161.4 (VDD), D162.4 (VDD), D163.4 (VDD), D164.4 (VDD), D17.4 (VDD), D18.4 (VDD), D19.4 (VDD), D2.4 (VDD), D20.4 (VDD), D21.4 (VDD), D22.4 (VDD), D23.4 (VDD), D24.4 (VDD), D25.4 (VDD), D26.4 (VDD), D27.4 (VDD), D28.4 (VDD), D29.4 (VDD), D3.4 (VDD), D30.4 (VDD), D31.4 (VDD), D32.4 (VDD), D33.4 (VDD), D34.4 (VDD), D35.4 (VDD), D36.4 (VDD), D37.4 (VDD), D38.4 (VDD), D39.4 (VDD), D4.4 (VDD), D40.4 (VDD), D41.4 (VDD), D42.4 (VDD), D43.4 (VDD), D44.4 (VDD), D45.4 (VDD), D46.4 (VDD), D47.4 (VDD), D48.4 (VDD), D49.4 (VDD), D5.4 (VDD), D50.4 (VDD), D51.4 (VDD), D52.4 (VDD), D53.4 (VDD), D54.4 (VDD), D55.4 (VDD), D56.4 (VDD), D57.4 (VDD), D58.4 (VDD), D59.4 (VDD), D6.4 (VDD), D60.4 (VDD), D61.4 (VDD), D62.4 (VDD), D63.4 (VDD), D64.4 (VDD), D65.4 (VDD), D66.4 (VDD), D67.4 (VDD), D68.4 (VDD), D69.4 (VDD), D7.4 (VDD), D70.4 (VDD), D71.4 (VDD), D72.4 (VDD), D73.4 (VDD), D74.4 (VDD), D75.4 (VDD), D76.4 (VDD), D77.4 (VDD), D78.4 (VDD), D79.4 (VDD), D8.4 (VDD), D80.4 (VDD), D81.4 (VDD), D82.4 (VDD), D83.4 (VDD), D84.4 (VDD), D85.4 (VDD), D86.4 (VDD), D87.4 (VDD), D88.4 (VDD), D89.4 (VDD), D9.4 (VDD), D90.4 (VDD), D91.4 (VDD), D92.4 (VDD), D93.4 (VDD), D94.4 (VDD), D95.4 (VDD), D96.4 (VDD), D97.4 (VDD), D98.4 (VDD), D99.4 (VDD)
- net GND: now also D1.2 (VSS), D10.2 (VSS), D100.2 (VSS), D101.2 (VSS), D102.2 (VSS), D103.2 (VSS), D104.2 (VSS), D105.2 (VSS), D106.2 (VSS), D107.2 (VSS), D108.2 (VSS), D109.2 (VSS), D11.2 (VSS), D110.2 (VSS), D111.2 (VSS), D112.2 (VSS), D113.2 (VSS), D114.2 (VSS), D115.2 (VSS), D116.2 (VSS), D117.2 (VSS), D118.2 (VSS), D119.2 (VSS), D12.2 (VSS), D120.2 (VSS), D121.2 (VSS), D122.2 (VSS), D123.2 (VSS), D124.2 (VSS), D125.2 (VSS), D126.2 (VSS), D127.2 (VSS), D128.2 (VSS), D129.2 (VSS), D13.2 (VSS), D130.2 (VSS), D131.2 (VSS), D132.2 (VSS), D133.2 (VSS), D134.2 (VSS), D135.2 (VSS), D136.2 (VSS), D137.2 (VSS), D138.2 (VSS), D139.2 (VSS), D14.2 (VSS), D140.2 (VSS), D141.2 (VSS), D142.2 (VSS), D143.2 (VSS), D144.2 (VSS), D145.2 (VSS), D146.2 (VSS), D147.2 (VSS), D148.2 (VSS), D149.2 (VSS), D15.2 (VSS), D150.2 (VSS), D151.2 (VSS), D152.2 (VSS), D153.2 (VSS), D154.2 (VSS), D155.2 (VSS), D156.2 (VSS), D157.2 (VSS), D158.2 (VSS), D159.2 (VSS), D16.2 (VSS), D160.2 (VSS), D161.2 (VSS), D162.2 (VSS), D163.2 (VSS), D164.2 (VSS), D17.2 (VSS), D18.2 (VSS), D19.2 (VSS), D2.2 (VSS), D20.2 (VSS), D21.2 (VSS), D22.2 (VSS), D23.2 (VSS), D24.2 (VSS), D25.2 (VSS), D26.2 (VSS), D27.2 (VSS), D28.2 (VSS), D29.2 (VSS), D3.2 (VSS), D30.2 (VSS), D31.2 (VSS), D32.2 (VSS), D33.2 (VSS), D34.2 (VSS), D35.2 (VSS), D36.2 (VSS), D37.2 (VSS), D38.2 (VSS), D39.2 (VSS), D4.2 (VSS), D40.2 (VSS), D41.2 (VSS), D42.2 (VSS), D43.2 (VSS), D44.2 (VSS), D45.2 (VSS), D46.2 (VSS), D47.2 (VSS), D48.2 (VSS), D49.2 (VSS), D5.2 (VSS), D50.2 (VSS), D51.2 (VSS), D52.2 (VSS), D53.2 (VSS), D54.2 (VSS), D55.2 (VSS), D56.2 (VSS), D57.2 (VSS), D58.2 (VSS), D59.2 (VSS), D6.2 (VSS), D60.2 (VSS), D61.2 (VSS), D62.2 (VSS), D63.2 (VSS), D64.2 (VSS), D65.2 (VSS), D66.2 (VSS), D67.2 (VSS), D68.2 (VSS), D69.2 (VSS), D7.2 (VSS), D70.2 (VSS), D71.2 (VSS), D72.2 (VSS), D73.2 (VSS), D74.2 (VSS), D75.2 (VSS), D76.2 (VSS), D77.2 (VSS), D78.2 (VSS), D79.2 (VSS), D8.2 (VSS), D80.2 (VSS), D81.2 (VSS), D82.2 (VSS), D83.2 (VSS), D84.2 (VSS), D85.2 (VSS), D86.2 (VSS), D87.2 (VSS), D88.2 (VSS), D89.2 (VSS), D9.2 (VSS), D90.2 (VSS), D91.2 (VSS), D92.2 (VSS), D93.2 (VSS), D94.2 (VSS), D95.2 (VSS), D96.2 (VSS), D97.2 (VSS), D98.2 (VSS), D99.2 (VSS)
- net LED: now also D1.3 (DIN)
- new net: D20.1 (DOUT), D21.3 (DIN)
- new net: D19.1 (DOUT), D20.3 (DIN)
- new net: D153.1 (DOUT), D154.3 (DIN)
- new net: D152.1 (DOUT), D153.3 (DIN)
- new net: D111.1 (DOUT), D112.3 (DIN)
- new net: D110.1 (DOUT), D111.3 (DIN)
- new net: D55.1 (DOUT), D56.3 (DIN)
- new net: D54.1 (DOUT), D55.3 (DIN)
- new net: D141.1 (DOUT), D142.3 (DIN)
- new net: D140.1 (DOUT), D141.3 (DIN)
- new net: D98.1 (DOUT), D99.3 (DIN)
- new net: D97.1 (DOUT), D98.3 (DIN)
- new net: D16.1 (DOUT), D17.3 (DIN)
- new net: D15.1 (DOUT), D16.3 (DIN)
- new net: D137.1 (DOUT), D138.3 (DIN)
- new net: D136.1 (DOUT), D137.3 (DIN)
- new net: D34.1 (DOUT), D35.3 (DIN)
- new net: D33.1 (DOUT), D34.3 (DIN)
- new net: D52.1 (DOUT), D53.3 (DIN)
- new net: D51.1 (DOUT), D52.3 (DIN)
- new net: D47.1 (DOUT), D48.3 (DIN)
- new net: D46.1 (DOUT), D47.3 (DIN)
- new net: D129.1 (DOUT), D130.3 (DIN)
- new net: D128.1 (DOUT), D129.3 (DIN)
- new net: D12.1 (DOUT), D13.3 (DIN)
- new net: D11.1 (DOUT), D12.3 (DIN)
- new net: D84.1 (DOUT), D85.3 (DIN)
- new net: D83.1 (DOUT), D84.3 (DIN)
- new net: D30.1 (DOUT), D31.3 (DIN)
- new net: D29.1 (DOUT), D30.3 (DIN)
- new net: D117.1 (DOUT), D118.3 (DIN)
- new net: D116.1 (DOUT), D117.3 (DIN)
- new net: D73.1 (DOUT), D74.3 (DIN)
- new net: D72.1 (DOUT), D73.3 (DIN)
- new net: D144.1 (DOUT), D145.3 (DIN)
- new net: D143.1 (DOUT), D144.3 (DIN)
- new net: D101.1 (DOUT), D102.3 (DIN)
- new net: D100.1 (DOUT), D101.3 (DIN)
- new net: D28.1 (DOUT), D29.3 (DIN)
- new net: D50.1 (DOUT), D51.3 (DIN)
- new net: D89.1 (DOUT), D90.3 (DIN)
- new net: D88.1 (DOUT), D89.3 (DIN)
- new net: D158.1 (DOUT), D159.3 (DIN)
- new net: D157.1 (DOUT), D158.3 (DIN)
- new net: D93.1 (DOUT), D94.3 (DIN)
- new net: D92.1 (DOUT), D93.3 (DIN)
- new net: D64.1 (DOUT), D65.3 (DIN)
- new net: D63.1 (DOUT), D64.3 (DIN)
- new net: D53.1 (DOUT), D54.3 (DIN)
- new net: D45.1 (DOUT), D46.3 (DIN)
- new net: D85.1 (DOUT), D86.3 (DIN)
- new net: D109.1 (DOUT), D110.3 (DIN)
- new net: D96.1 (DOUT), D97.3 (DIN)
- new net: D135.1 (DOUT), D136.3 (DIN)
- new net: D134.1 (DOUT), D135.3 (DIN)
- new net: D3.1 (DOUT), D4.3 (DIN)
- new net: D2.1 (DOUT), D3.3 (DIN)
- new net: D161.1 (DOUT), D162.3 (DIN)
- new net: D160.1 (DOUT), D161.3 (DIN)
- new net: D31.1 (DOUT), D32.3 (DIN)
- new net: D68.1 (DOUT), D69.3 (DIN)
- new net: D67.1 (DOUT), D68.3 (DIN)
- new net: D139.1 (DOUT), D140.3 (DIN)
- new net: D138.1 (DOUT), D139.3 (DIN)
- new net: D123.1 (DOUT), D124.3 (DIN)
- new net: D122.1 (DOUT), D123.3 (DIN)
- new net: D82.1 (DOUT), D83.3 (DIN)
- new net: D133.1 (DOUT), D134.3 (DIN)
- new net: D132.1 (DOUT), D133.3 (DIN)
- new net: D100.3 (DIN), D99.1 (DOUT)
- new net: D69.1 (DOUT), D70.3 (DIN)
- new net: D162.1 (DOUT), D163.3 (DIN)
- new net: D65.1 (DOUT), D66.3 (DIN)
- new net: D62.1 (DOUT), D63.3 (DIN)
- new net: D44.1 (DOUT), D45.3 (DIN)
- new net: D43.1 (DOUT), D44.3 (DIN)
- new net: D127.1 (DOUT), D128.3 (DIN)
- new net: D126.1 (DOUT), D127.3 (DIN)
- new net: D42.1 (DOUT), D43.3 (DIN)
- new net: D94.1 (DOUT), D95.3 (DIN)
- new net: D59.1 (DOUT), D60.3 (DIN)
- new net: D58.1 (DOUT), D59.3 (DIN)
- new net: D61.1 (DOUT), D62.3 (DIN)
- new net: D18.1 (DOUT), D19.3 (DIN)
- new net: D21.1 (DOUT), D22.3 (DIN)
- new net: D114.1 (DOUT), D115.3 (DIN)
- new net: D113.1 (DOUT), D114.3 (DIN)
- new net: D24.1 (DOUT), D25.3 (DIN)
- new net: D23.1 (DOUT), D24.3 (DIN)
- new net: D66.1 (DOUT), D67.3 (DIN)
- new net: D108.1 (DOUT), D109.3 (DIN)
- new net: D107.1 (DOUT), D108.3 (DIN)
- new net: D76.1 (DOUT), D77.3 (DIN)
- new net: D75.1 (DOUT), D76.3 (DIN)
- new net: D147.1 (DOUT), D148.3 (DIN)
- new net: D146.1 (DOUT), D147.3 (DIN)
- new net: D151.1 (DOUT), D152.3 (DIN)
- new net: D150.1 (DOUT), D151.3 (DIN)
- new net: D120.1 (DOUT), D121.3 (DIN)
- new net: D119.1 (DOUT), D120.3 (DIN)
- new net: D22.1 (DOUT), D23.3 (DIN)
- new net: D121.1 (DOUT), D122.3 (DIN)
- new net: D124.1 (DOUT), D125.3 (DIN)
- new net: D56.1 (DOUT), D57.3 (DIN)
- new net: D38.1 (DOUT), D39.3 (DIN)
- new net: D37.1 (DOUT), D38.3 (DIN)
- new net: D142.1 (DOUT), D143.3 (DIN)
- new net: D131.1 (DOUT), D132.3 (DIN)
- new net: D130.1 (DOUT), D131.3 (DIN)
- new net: D115.1 (DOUT), D116.3 (DIN)
- new net: D26.1 (DOUT), D27.3 (DIN)
- new net: D25.1 (DOUT), D26.3 (DIN)
- new net: D81.1 (DOUT), D82.3 (DIN)
- new net: D77.1 (DOUT), D78.3 (DIN)
- new net: D154.1 (DOUT), D155.3 (DIN)
- new net: D78.1 (DOUT), D79.3 (DIN)
- new net: D32.1 (DOUT), D33.3 (DIN)
- new net: D70.1 (DOUT), D71.3 (DIN)
- new net: D60.1 (DOUT), D61.3 (DIN)
- new net: D57.1 (DOUT), D58.3 (DIN)
- new net: D36.1 (DOUT), D37.3 (DIN)
- new net: D35.1 (DOUT), D36.3 (DIN)
- new net: D87.1 (DOUT), D88.3 (DIN)
- new net: D13.1 (DOUT), D14.3 (DIN)
- new net: D86.1 (DOUT), D87.3 (DIN)
- new net: D112.1 (DOUT), D113.3 (DIN)
- new net: D79.1 (DOUT), D80.3 (DIN)
- new net: D40.1 (DOUT), D41.3 (DIN)
- new net: D39.1 (DOUT), D40.3 (DIN)
- new net: D6.1 (DOUT), D7.3 (DIN)
- new net: D5.1 (DOUT), D6.3 (DIN)
- new net: D1.1 (DOUT), D2.3 (DIN)
- new net: D104.1 (DOUT), D105.3 (DIN)
- new net: D103.1 (DOUT), D104.3 (DIN)
- new net: D148.1 (DOUT), D149.3 (DIN)
- new net: D156.1 (DOUT), D157.3 (DIN)
- new net: D163.1 (DOUT), D164.3 (DIN)
- new net: D14.1 (DOUT), D15.3 (DIN)
- new net: D8.1 (DOUT), D9.3 (DIN)
- new net: D7.1 (DOUT), D8.3 (DIN)
- new net: D145.1 (DOUT), D146.3 (DIN)
- new net: D17.1 (DOUT), D18.3 (DIN)
- new net: D27.1 (DOUT), D28.3 (DIN)
- new net: D91.1 (DOUT), D92.3 (DIN)
- new net: D90.1 (DOUT), D91.3 (DIN)
- new net: D95.1 (DOUT), D96.3 (DIN)
- new net: D155.1 (DOUT), D156.3 (DIN)
- new net: D71.1 (DOUT), D72.3 (DIN)
- new net: D74.1 (DOUT), D75.3 (DIN)
- new net: D106.1 (DOUT), D107.3 (DIN)
- new net: D102.1 (DOUT), D103.3 (DIN)
- new net: D48.1 (DOUT), D49.3 (DIN)
- new net: D118.1 (DOUT), D119.3 (DIN)
- new net: D4.1 (DOUT), D5.3 (DIN)
- new net: D159.1 (DOUT), D160.3 (DIN)
- new net: D10.3 (DIN), D9.1 (DOUT)
- new net: D125.1 (DOUT), D126.3 (DIN)
- new net: D41.1 (DOUT), D42.3 (DIN)
- new net: D49.1 (DOUT), D50.3 (DIN)
- new net: D80.1 (DOUT), D81.3 (DIN)
- new net: D10.1 (DOUT), D11.3 (DIN)
- new net: D105.1 (DOUT), D106.3 (DIN)
- new net: D149.1 (DOUT), D150.3 (DIN)
