File: buttonMatrixBoard/buttonMatrixBoard.kicad_sch (KiCad schematic)
At the start: 42 parts, among them J1 Conn_01x04_Pin, J2 Conn_01x02_Pin, J3 Conn_01x02_Pin, J4 Conn_01x04_Pin, J5 Conn_01x04_Pin, J6 Conn_01x03_Pin, SW1 SW_Push, SW2 SW_Push, SW3 SW_Push, SW4 SW_Push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

Commit message: buttonMatrix changed Diode footprint
Parts:
- D1, D2, D3, D4, D5, D6, D7, D8: footprint Diode_SMD:D_SOD-323 -> Diode_SMD:D_SOD-323_HandSoldering
Changed lines of the file:
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@@
       (effects (font (size 1.27 1.27)))
     )
-    (property "Footprint" "Diode_SMD:D_SOD-323" (at 73.66 50.165 0)
+    (property "Footprint" "Diode_SMD:D_SOD-323_HandSoldering" (at 73.66 50.165 0)
       (effects (font (size 1.27 1.27)) hide)
     )
@@
       (effects (font (size 1.27 1.27)))
     )
-    (property "Footprint" "Diode_SMD:D_SOD-323" (at 121.92 50.165 0)
+    (property "Footprint" "Diode_SMD:D_SOD-323_HandSoldering" (at 121.92 50.165 0)
       (effects (font (size 1.27 1.27)) hide)
     )
@@
       (effects (font (size 1.27 1.27)))
     )
-    (property "Footprint" "Diode_SMD:D_SOD-323" (at 97.79 50.165 0)
+    (property "Footprint" "Diode_SMD:D_SOD-323_HandSoldering" (at 97.79 50.165 0)
       (effects (font (size 1.27 1.27)) hide)
     )
@@
       (effects (font (size 1.27 1.27)))
     )
-    (property "Footprint" "Diode_SMD:D_SOD-323" (at 121.92 65.405 0)
+    (property "Footprint" "Diode_SMD:D_SOD-323_HandSoldering" (at 121.92 65.405 0)
       (effects (font (size 1.27 1.27)) hide)
     )
@@
       (effects (font (size 1.27 1.27)))
     )
-    (property "Footprint" "Diode_SMD:D_SOD-323" (at 97.79 65.405 0)
+    (property "Footprint" "Diode_SMD:D_SOD-323_HandSoldering" (at 97.79 65.405 0)
       (effects (font (size 1.27 1.27)) hide)
     )
@@
       (effects (font (size 1.27 1.27)))
     )
-    (property "Footprint" "Diode_SMD:D_SOD-323" (at 73.66 65.405 0)
+    (property "Footprint" "Diode_SMD:D_SOD-323_HandSoldering" (at 73.66 65.405 0)
       (effects (font (size 1.27 1.27)) hide)
     )
@@
       (effects (font (size 1.27 1.27)))
     )
-    (property "Footprint" "Diode_SMD:D_SOD-323" (at 49.53 65.405 0)
+    (property "Footprint" "Diode_SMD:D_SOD-323_HandSoldering" (at 49.53 65.405 0)
       (effects (font (size 1.27 1.27)) hide)
     )
@@
       (effects (font (size 1.27 1.27)))
     )
-    (property "Footprint" "Diode_SMD:D_SOD-323" (at 49.53 50.165 0)
-      (effects (font (size 1.27 1.27)) hide)
-    )
+    (property "Footprint" "Diode_SMD:D_SOD-323_HandSoldering" (at 49.53 50.165 0)
+      (effects (font (size 1.27 1.27)) hide)
+    )
