File: CAT_XLR/CAT_XLR.kicad_pcb (KiCad board)
At the start: 2 copper layers, 46 x 120 mm, 26 parts, among them J0 8P8C_Shielded, J1 XLR5, J2 XLR5, J3 XLR5, J4 XLR5, J5 XLR5, J6 XLR5, J7 XLR5, J8 XLR5

Commit message: fixed CAT connection and gnd connection
Parts:
- renumbered REF** to ?
Connections:
- J0 pad 4: DATA- 2 -> DATA- 3
- J0 pad 6: DATA- 3 -> DATA- 2
- J1 pad G: (no net) -> GND
- J2 pad G: (no net) -> GND
- J3 pad G: (no net) -> GND
- J4 pad G: (no net) -> GND
- J5 pad G: (no net) -> GND
- J6 pad G: (no net) -> GND
- J7 pad G: (no net) -> GND
- J8 pad G: (no net) -> GND
Routing:
- net DATA- 2: track 77.2 -> 78.4 mm
- net DATA+ 3: track 79.7 -> 80.0 mm, vias 1 -> 2
- net DATA- 3: track 102.4 -> 102.7 mm, vias 1 -> 2
