File: motorFaderBoard/motorFaderBoard.kicad_pcb (KiCad board)
At the start: 2 copper layers, 42 x 100 mm, 17 parts, among them J1 Conn_01x04_Pin, J2 Conn_01x04_Pin, J3 Conn_01x04_Socket, J4 Conn_01x04_Socket, J5 Conn_01x15_Socket, J6 Conn_01x15_Socket, J7 Conn_01x06_Socket, J8 Conn_01x03_Socket, J9 Conn_01x03_Pin, U3 L293DD

Commit message: connectors, labels, vias
Parts:
- removed the J2 at (40.0, 16.2)
- removed the J9 at (40.0, 70.0)
- added J3: Conn_01x04_Pin, Connector_PinHeader_2.54mm:PinHeader_1x04_P2.54mm_Vertical, B.Cu at (-20.0, 35.0)
- added J5: Conn_01x03_Pin, Connector_PinHeader_2.54mm:PinHeader_1x03_P2.54mm_Vertical, B.Cu at (2.00, 72.0)
- J9: renamed from J7; footprint Connector_PinSocket_2.54mm:PinSocket_1x05_P2.54mm_Vertical -> Connector_PinSocket_2.54mm:PinSocket_1x06_P2.54mm_Vertical
- moved J2 53.5 mm to (40.0, 16.0)
- moved J6 38.1 mm to (40.0, 72.0)
- moved J4 3.38 mm to (-15.0, 35.0)
- moved J9 1.00 mm to (40.0, 54.8)
- moved U1 0.22 mm to (21.0, 83.0)
- moved J1 0.19 mm to (2.00, 16.0)
- renumbered J3 to J2, J8 to J6, J5 to J7, J6 to J8, U3 to U1
Connections:
- A1 pad 16: unconnected-(A1-D13-Pad16) -> XD13
- A1 pad 17: unconnected-(A1-3V3-Pad17) -> X3V3
- A1 pad 19: unconnected-(A1-A0-Pad19) -> XA0
- A1 pad 20: unconnected-(A1-A1-Pad20) -> XA1
- A1 pad 21: unconnected-(A1-A2-Pad21) -> XA2
- A1 pad 22: unconnected-(A1-A3-Pad22) -> XA3
- A1 pad 28: unconnected-(A1-~{RESET}-Pad28) -> XRST2
- A1 pad 3: unconnected-(A1-~{RESET}-Pad3) -> XRST
- A1 pad 30: unconnected-(A1-VIN-Pad30) -> XVIN
- A1 pad 5: unconnected-(A1-D2-Pad5) -> XD2
- J7 pad 3: unconnected-(J5-Pin_3-Pad3) -> XRST
- J7 pad 5: unconnected-(J5-Pin_5-Pad5) -> XD2
- J8 pad 1: unconnected-(J6-Pin_1-Pad1) -> XVIN
- J8 pad 10: unconnected-(J6-Pin_10-Pad10) -> XA2
- J8 pad 11: unconnected-(J6-Pin_11-Pad11) -> XA1
- J8 pad 12: unconnected-(J6-Pin_12-Pad12) -> XA0
- J8 pad 14: unconnected-(J6-Pin_14-Pad14) -> X3V3
- J8 pad 15: unconnected-(J6-Pin_15-Pad15) -> XD13
- J8 pad 3: unconnected-(J6-Pin_3-Pad3) -> XRST2
- J8 pad 9: unconnected-(J6-Pin_9-Pad9) -> XA3
Routing:
- net VCC: track 220.6 -> 226.7 mm
- net +9V: track 56.2 -> 54.4 mm, vias 3 -> 2
- net TX: track 10.4 -> 11.4 mm
- net RX: track 10.4 -> 11.4 mm
- net M2B_I: track 44.9 -> 45.9 mm
- net M1B_I: track 44.5 -> 45.3 mm
- net SDA: track 70.5 -> 71.1 mm
- net M1B: track 21.2 -> 21.7 mm
- net GND: vias 0 -> 11
- added copper zone on F.Cu, net GND
- removed copper zone on F.Cu, net (none)
Other:
- board text added: "+9V"
- board text added: "GND"
- board text added: "RX"
- board text added: "TX"
- board text added: "VCC"
